Commit message: Generic body offset calculated with wheel height

File: ros_ws/src/racer_model/racer_description/racer.xacro (robot description, xacro)
@@ -16,5 +16,5 @@
     <inertial>
       <mass value="${bodyMass}"/>
-      <origin xyz="0 0 0.05" rpy=" 0 0 0"/>
+      <origin xyz="0 0 ${wheel_height}/2" rpy=" 0 0 0"/>
       <box_inertia  m="${bodyMass}" l="${bodySizeL}" b="${bodySizeB}" h="${bodySizeH}" />
     </inertial>
@@ -25,5 +25,5 @@
     </collision>
     <visual name='chassis_visual'>
-      <origin xyz="0 0 0.05" rpy=" 0 0 0"/>
+      <origin xyz="0 0 ${wheel_height}/2" rpy=" 0 0 0"/>
       <geometry>
         <box size="${bodySizeL} ${bodySizeB} ${bodySizeH}"/>
@@ -43,9 +43,9 @@
     <inertial>
       <mass value="${cameraMass}" />
-      <origin xyz="0 0 0.05" rpy="0 0 0"/>
+      <origin xyz="0 0 ${wheel_height}/2" rpy="0 0 0"/>
       <box_inertia m="${cameraMass}" l="${cameraSize}" b="${cameraSize}" h="${cameraSize}" />
     </inertial>
     <collision>
-      <origin xyz="0.01 0 0.05" rpy="0 0 0"/>
+      <origin xyz="0 0 ${wheel_height}/2" rpy="0 0 0"/>
       <geometry>
         <box size="${cameraSize} ${cameraSize} ${cameraSize}"/>
@@ -53,5 +53,5 @@
     </collision>
     <visual>
-      <origin xyz="0.01 0 0.05" rpy="0 0 0"/>
+      <origin xyz="0 0 ${wheel_height}/2" rpy="0 0 0"/>
       <geometry>
         <box size="${cameraSize} ${cameraSize} ${cameraSize}"/>
@@ -72,9 +72,9 @@
     <inertial>
       <mass value="${hokuyoMass}" />
-      <origin xyz="0 0 0.05" rpy="0 0 0"/>
+      <origin xyz="0 0 ${wheel_height}/2" rpy="0 0 0"/>
       <box_inertia  m="${hokuyoMass}" l="${hokuyoSize}" b="${hokuyoSize}" h="${hokuyoSize}" />
     </inertial>
     <collision>
-      <origin xyz="0.01 0 0.05" rpy="0 0 0"/>
+      <origin xyz="0 0 ${wheel_height}/2" rpy="0 0 0"/>
       <geometry>
     	  <box size="${hokuyoSize} ${hokuyoSize} ${hokuyoSize}"/>
@@ -82,5 +82,5 @@
     </collision>
     <visual>
-      <origin xyz="0.01 0 0.05" rpy="0 0 0"/>
+      <origin xyz="0 0 ${wheel_height}/2" rpy="0 0 0"/>
       <geometry>
         <mesh filename="package://racer_model/racer_description/meshes/hokuyo.dae"/>

Commit message: Fixed collision boxes

File: ros_ws/src/racer_model/racer_description/racer.xacro (robot description, xacro)
@@ -20,4 +20,5 @@
     </inertial>
     <collision name='collision'>
+      <origin xyz="0 0 ${wheel_height}/2" rpy=" 0 0 0"/>
       <geometry>
         <box size="${bodySizeL} ${bodySizeB} ${bodySizeH}"/>

File: ros_ws/src/racer_model/racer_description/racer_macros.xacro (robot description, xacro)
@@ -27,5 +27,5 @@
       </inertial>
       <collision>
-        <origin xyz="0 ${OffsetY} 0" rpy="${flipY*pi/2} 0 0 " />
+        <origin xyz="0 ${OffsetY} 0" rpy="${flipY*pi/180} 0 0 " />
         <geometry>
           <cylinder length="${wheel_height}" radius="${wheel_radius}" />

Commit message: Fix math expressions in racer description

File: ros_ws/src/racer_model/racer_description/racer.xacro (robot description, xacro)
@@ -16,9 +16,9 @@
     <inertial>
       <mass value="${bodyMass}"/>
-      <origin xyz="0 0 ${wheel_height}/2" rpy=" 0 0 0"/>
+      <origin xyz="0 0 ${wheel_height/2}" rpy=" 0 0 0"/>
       <box_inertia  m="${bodyMass}" l="${bodySizeL}" b="${bodySizeB}" h="${bodySizeH}" />
     </inertial>
     <collision name='collision'>
-      <origin xyz="0 0 ${wheel_height}/2" rpy=" 0 0 0"/>
+      <origin xyz="0 0 ${wheel_height/2}" rpy=" 0 0 0"/>
       <geometry>
         <box size="${bodySizeL} ${bodySizeB} ${bodySizeH}"/>
@@ -26,5 +26,5 @@
     </collision>
     <visual name='chassis_visual'>
-      <origin xyz="0 0 ${wheel_height}/2" rpy=" 0 0 0"/>
+      <origin xyz="0 0 ${wheel_height/2}" rpy=" 0 0 0"/>
       <geometry>
         <box size="${bodySizeL} ${bodySizeB} ${bodySizeH}"/>
@@ -44,9 +44,9 @@
     <inertial>
       <mass value="${cameraMass}" />
-      <origin xyz="0 0 ${wheel_height}/2" rpy="0 0 0"/>
+      <origin xyz="0 0 ${wheel_height/2}" rpy="0 0 0"/>
       <box_inertia m="${cameraMass}" l="${cameraSize}" b="${cameraSize}" h="${cameraSize}" />
     </inertial>
     <collision>
-      <origin xyz="0 0 ${wheel_height}/2" rpy="0 0 0"/>
+      <origin xyz="0 0 ${wheel_height/2}" rpy="0 0 0"/>
       <geometry>
         <box size="${cameraSize} ${cameraSize} ${cameraSize}"/>
@@ -54,5 +54,5 @@
     </collision>
     <visual>
-      <origin xyz="0 0 ${wheel_height}/2" rpy="0 0 0"/>
+      <origin xyz="0 0 ${wheel_height/2}" rpy="0 0 0"/>
       <geometry>
         <box size="${cameraSize} ${cameraSize} ${cameraSize}"/>
@@ -73,9 +73,9 @@
     <inertial>
       <mass value="${hokuyoMass}" />
-      <origin xyz="0 0 ${wheel_height}/2" rpy="0 0 0"/>
+      <origin xyz="0 0 ${wheel_height/2}" rpy="0 0 0"/>
       <box_inertia  m="${hokuyoMass}" l="${hokuyoSize}" b="${hokuyoSize}" h="${hokuyoSize}" />
     </inertial>
     <collision>
-      <origin xyz="0 0 ${wheel_height}/2" rpy="0 0 0"/>
+      <origin xyz="0 0 ${wheel_height/2}" rpy="0 0 0"/>
       <geometry>
     	  <box size="${hokuyoSize} ${hokuyoSize} ${hokuyoSize}"/>
@@ -83,5 +83,5 @@
     </collision>
     <visual>
-      <origin xyz="0 0 ${wheel_height}/2" rpy="0 0 0"/>
+      <origin xyz="0 0 ${wheel_height/2}" rpy="0 0 0"/>
       <geometry>
         <mesh filename="package://racer_model/racer_description/meshes/hokuyo.dae"/>

Commit message: Fliped Intertials of Wheels

File: ros_ws/src/racer_model/racer_description/racer.xacro (robot description, xacro)
@@ -10,8 +10,7 @@
   <xacro:property name="bodySizeB" value="0.18"/>
   <xacro:property name="bodySizeH" value="0.1"/>
-  <xacro:property name="bodyMass" value="10"/>
+  <xacro:property name="bodyMass" value="3.5"/>
   <!--  Body  -->
   <link name='chassis'>
-    <pose>0 0 0.1 0 0 0</pose>
     <inertial>
       <mass value="${bodyMass}"/>

File: ros_ws/src/racer_model/racer_description/racer_macros.xacro (robot description, xacro)
@@ -15,5 +15,5 @@
   <property name="wheel_radius" value="0.05" />
   <property name="wheel_height" value="0.045" />
-  <property name="wheel_mass" value="2.5" />
+  <property name="wheel_mass" value="0.2" />
   <property name="base_x_origin_to_wheel_origin" value="0.16" />
   <property name="base_y_origin_to_wheel_origin" value="0.095" />
@@ -23,5 +23,5 @@
       <inertial>
         <mass value="${wheel_mass}" />
-        <origin xyz="0 ${OffsetY} 0" />
+        <origin xyz="0 ${OffsetY} 0" rpy="${flipY*pi/180} 0  0 "/>
         <cylinder_inertia  m="${wheel_mass}" r="${wheel_radius}" h="${wheel_height}" />
       </inertial>

Commit message: Add 3D model for the car in gazebo

File: ros_ws/src/racer_model/racer_description/racer.xacro (robot description, xacro)
@@ -24,19 +24,16 @@
       </geometry>
     </collision>
-    <visual name='chassis_visual'>
-      <origin xyz="0 0 ${wheel_height/2}" rpy=" 0 0 0"/>
+    <visual>
+      <origin xyz="0 0 0" rpy="0 0 0"/>
       <geometry>
-        <box size="${bodySizeL} ${bodySizeB} ${bodySizeH}"/>
+        <mesh filename="package://racer_model/racer_description/meshes/car.dae"/>
       </geometry>
     </visual>
   </link>
-  <gazebo reference="chassis">
-    <material>Gazebo/Green</material>
-  </gazebo>
   <!--  Wheels  -->
-  <wheel  fb="front" lr="left" parent="chassis" translateX="1" translateY="1" flipY="90" OffsetY="0.02" />
-  <wheel  fb="back" lr="left" parent="chassis" translateX="-1" translateY="1" flipY="90" OffsetY="0.02" />
-  <wheel  fb="front" lr="right" parent="chassis" translateX="1" translateY="-1" flipY="90" OffsetY="-0.02" />
-  <wheel  fb="back" lr="right" parent="chassis" translateX="-1" translateY="-1" flipY="90" OffsetY="-0.02" />
+  <wheel  fb="front" lr="left" parent="chassis" translateX="1" translateY="1" left="1" OffsetY="0.02" />
+  <wheel  fb="back" lr="left" parent="chassis" translateX="-1" translateY="1" left="1" OffsetY="0.02" />
+  <wheel  fb="front" lr="right" parent="chassis" translateX="1" translateY="-1" left="0" OffsetY="-0.02" />
+  <wheel  fb="back" lr="right" parent="chassis" translateX="-1" translateY="-1" left="0" OffsetY="-0.02" />
   <!-- Camera -->
   <link name="camera">

File: ros_ws/src/racer_model/racer_description/racer_macros.xacro (robot description, xacro)
@@ -19,27 +19,24 @@
   <property name="base_y_origin_to_wheel_origin" value="0.095" />
   <property name="base_z_origin_to_wheel_origin" value="0" />
-  <xacro:macro name="wheel" params="fb lr parent translateX translateY flipY OffsetY">
+  <xacro:macro name="wheel" params="fb lr parent translateX translateY left OffsetY">
     <link name="${lr}_wheel_${fb}">
       <inertial>
         <mass value="${wheel_mass}" />
-        <origin xyz="0 ${OffsetY} 0" rpy="${flipY*pi/180} 0  0 "/>
+        <origin xyz="0 ${OffsetY} 0" rpy="${90*pi/180} 0 0"/>
         <cylinder_inertia  m="${wheel_mass}" r="${wheel_radius}" h="${wheel_height}" />
       </inertial>
       <collision>
-        <origin xyz="0 ${OffsetY} 0" rpy="${flipY*pi/180} 0 0 " />
+        <origin xyz="0 ${OffsetY} 0" rpy="${90*pi/180} 0 0 " />
         <geometry>
           <cylinder length="${wheel_height}" radius="${wheel_radius}" />
         </geometry>
       </collision>
-      <visual>
-        <origin xyz="0 ${OffsetY} 0" rpy="${flipY*pi/180} 0  0 " />
-        <geometry>
-          <cylinder length="${wheel_height}" radius="${wheel_radius}" />
-        </geometry>
+      <visual name="visual">
+          <origin xyz="0 ${OffsetY} 0" rpy="0 0 ${left*pi}" />
+          <geometry>
+            <mesh filename="package://racer_model/racer_description/meshes/wheel.dae"/>
+          </geometry>
       </visual>
     </link>
-    <gazebo reference="${lr}_wheel_${fb}">
-      <material>Gazebo/Black</material>
-    </gazebo>
     <joint name="${lr}_wheel_${fb}_hinge" type="continuous">
       <parent link="${parent}"/>

Commit message: Add model for the ZED camera

File: ros_ws/src/racer_model/racer_description/racer.xacro (robot description, xacro)
@@ -3,5 +3,4 @@
   <xacro:include filename="$(find racer_model)/racer_description/racer_plugins.gazebo" />
   <xacro:include filename="$(find racer_model)/racer_description/racer_macros.xacro" />
-  <xacro:property name="cameraSize" value="0.05"/>
   <xacro:property name="cameraMass" value="0.1"/>
   <xacro:property name="hokuyoSize" value="0.1"/>
@@ -41,22 +40,19 @@
       <mass value="${cameraMass}" />
       <origin xyz="0 0 ${wheel_height/2}" rpy="0 0 0"/>
-      <box_inertia m="${cameraMass}" l="${cameraSize}" b="${cameraSize}" h="${cameraSize}" />
+      <box_inertia m="${cameraMass}" l="0.03" b="0.03" h="0.17" />
     </inertial>
     <collision>
       <origin xyz="0 0 ${wheel_height/2}" rpy="0 0 0"/>
       <geometry>
-        <box size="${cameraSize} ${cameraSize} ${cameraSize}"/>
+        <box size="0.03 0.17 0.03"/>
       </geometry>
     </collision>
     <visual>
-      <origin xyz="0 0 ${wheel_height/2}" rpy="0 0 0"/>
+      <origin xyz="0 0 0" rpy="0 0 0"/>
       <geometry>
-        <box size="${cameraSize} ${cameraSize} ${cameraSize}"/>
+        <mesh filename="package://racer_model/racer_description/meshes/ZED.dae"/>
       </geometry>
     </visual>
   </link>
-  <gazebo reference="camera">
-    <material>Gazebo/Red</material>
-  </gazebo>
   <joint name="camera_joint" type="fixed">
     <axis xyz="0 1 0" />

Commit message: Add 3D model for the car in gazebo (#77)
* Add 3D model for the car in gazebo

* Add model for the ZED camera

File: ros_ws/src/racer_model/racer_description/racer.xacro (robot description, xacro)
@@ -3,5 +3,4 @@
   <xacro:include filename="$(find racer_model)/racer_description/racer_plugins.gazebo" />
   <xacro:include filename="$(find racer_model)/racer_description/racer_macros.xacro" />
-  <xacro:property name="cameraSize" value="0.05"/>
   <xacro:property name="cameraMass" value="0.1"/>
   <xacro:property name="hokuyoSize" value="0.1"/>
@@ -24,19 +23,16 @@
       </geometry>
     </collision>
-    <visual name='chassis_visual'>
-      <origin xyz="0 0 ${wheel_height/2}" rpy=" 0 0 0"/>
+    <visual>
+      <origin xyz="0 0 0" rpy="0 0 0"/>
       <geometry>
-        <box size="${bodySizeL} ${bodySizeB} ${bodySizeH}"/>
+        <mesh filename="package://racer_model/racer_description/meshes/car.dae"/>
       </geometry>
     </visual>
   </link>
-  <gazebo reference="chassis">
-    <material>Gazebo/Green</material>
-  </gazebo>
   <!--  Wheels  -->
-  <wheel  fb="front" lr="left" parent="chassis" translateX="1" translateY="1" flipY="90" OffsetY="0.02" />
-  <wheel  fb="back" lr="left" parent="chassis" translateX="-1" translateY="1" flipY="90" OffsetY="0.02" />
-  <wheel  fb="front" lr="right" parent="chassis" translateX="1" translateY="-1" flipY="90" OffsetY="-0.02" />
-  <wheel  fb="back" lr="right" parent="chassis" translateX="-1" translateY="-1" flipY="90" OffsetY="-0.02" />
+  <wheel  fb="front" lr="left" parent="chassis" translateX="1" translateY="1" left="1" OffsetY="0.02" />
+  <wheel  fb="back" lr="left" parent="chassis" translateX="-1" translateY="1" left="1" OffsetY="0.02" />
+  <wheel  fb="front" lr="right" parent="chassis" translateX="1" translateY="-1" left="0" OffsetY="-0.02" />
+  <wheel  fb="back" lr="right" parent="chassis" translateX="-1" translateY="-1" left="0" OffsetY="-0.02" />
   <!-- Camera -->
   <link name="camera">
@@ -44,22 +40,19 @@
       <mass value="${cameraMass}" />
       <origin xyz="0 0 ${wheel_height/2}" rpy="0 0 0"/>
-      <box_inertia m="${cameraMass}" l="${cameraSize}" b="${cameraSize}" h="${cameraSize}" />
+      <box_inertia m="${cameraMass}" l="0.03" b="0.03" h="0.17" />
     </inertial>
     <collision>
       <origin xyz="0 0 ${wheel_height/2}" rpy="0 0 0"/>
       <geometry>
-        <box size="${cameraSize} ${cameraSize} ${cameraSize}"/>
+        <box size="0.03 0.17 0.03"/>
       </geometry>
     </collision>
     <visual>
-      <origin xyz="0 0 ${wheel_height/2}" rpy="0 0 0"/>
+      <origin xyz="0 0 0" rpy="0 0 0"/>
       <geometry>
-        <box size="${cameraSize} ${cameraSize} ${cameraSize}"/>
+        <mesh filename="package://racer_model/racer_description/meshes/ZED.dae"/>
       </geometry>
     </visual>
   </link>
-  <gazebo reference="camera">
-    <material>Gazebo/Red</material>
-  </gazebo>
   <joint name="camera_joint" type="fixed">
     <axis xyz="0 1 0" />
