Commit message: Exchanged Diff. Drive by ros_control plugin

File: ros_ws/src/racer_model/racer_description/urdf/racer.xacro (robot description, xacro)
@@ -1,6 +1,7 @@
 <?xml version='1.0'?>
 <robot name="myrobot" xmlns:xacro="http://www.ros.org/wiki/xacro">
-  <xacro:include filename="$(find racer_model)/racer_description/racer_plugins.gazebo" />
-  <xacro:include filename="$(find racer_model)/racer_description/racer_macros.xacro" />
+  <xacro:include filename="$(find racer_model)/racer_description/urdf/racer_plugins.gazebo" />
+  <xacro:include filename="$(find racer_model)/racer_description/urdf/racer_macros.xacro" />
+  <xacro:property name="cameraSize" value="0.05"/>
   <xacro:property name="cameraMass" value="0.1"/>
   <xacro:property name="hokuyoSize" value="0.1"/>
@@ -23,16 +24,22 @@
       </geometry>
     </collision>
-    <visual>
-      <origin xyz="0 0 0" rpy="0 0 0"/>
+    <visual name='chassis_visual'>
+      <origin xyz="0 0 ${wheel_height/2}" rpy=" 0 0 0"/>
       <geometry>
-        <mesh filename="package://racer_model/racer_description/meshes/car.dae"/>
+        <box size="${bodySizeL} ${bodySizeB} ${bodySizeH}"/>
       </geometry>
     </visual>
   </link>
+  <gazebo reference="chassis">
+    <material>Gazebo/Green</material>
+  </gazebo>
   <!--  Wheels  -->
-  <wheel  fb="front" lr="left" parent="chassis" translateX="1" translateY="1" left="1" OffsetY="0.02" />
-  <wheel  fb="back" lr="left" parent="chassis" translateX="-1" translateY="1" left="1" OffsetY="0.02" />
-  <wheel  fb="front" lr="right" parent="chassis" translateX="1" translateY="-1" left="0" OffsetY="-0.02" />
-  <wheel  fb="back" lr="right" parent="chassis" translateX="-1" translateY="-1" left="0" OffsetY="-0.02" />
+  <wheel  fb="front" lr="left" parent="chassis" translateX="1" translateY="1" flip="90" OffsetY="0.035" />
+  <wheel  fb="back" lr="left" parent="chassis" translateX="-1" translateY="1" flip="90" OffsetY="0.035" />
+  <wheel  fb="front" lr="right" parent="chassis" translateX="1" translateY="-1" flip="90" OffsetY="-0.035" />
+  <wheel  fb="back" lr="right" parent="chassis" translateX="-1" translateY="-1" flip="90" OffsetY="-0.035" />
+  <!-- Steering -->
+  <steering_hinge  lr="left" parent="chassis" translateY="1" OffsetY="0.01" />
+  <steering_hinge  lr="right" parent="chassis" translateY="-1" OffsetY="-0.01" />
   <!-- Camera -->
   <link name="camera">
@@ -40,19 +47,22 @@
       <mass value="${cameraMass}" />
       <origin xyz="0 0 ${wheel_height/2}" rpy="0 0 0"/>
-      <box_inertia m="${cameraMass}" l="0.03" b="0.03" h="0.17" />
+      <box_inertia m="${cameraMass}" l="${cameraSize}" b="${cameraSize}" h="${cameraSize}" />
     </inertial>
     <collision>
       <origin xyz="0 0 ${wheel_height/2}" rpy="0 0 0"/>
       <geometry>
-        <box size="0.03 0.17 0.03"/>
+        <box size="${cameraSize} ${cameraSize} ${cameraSize}"/>
       </geometry>
     </collision>
     <visual>
-      <origin xyz="0 0 0" rpy="0 0 0"/>
+      <origin xyz="0 0 ${wheel_height/2}" rpy="0 0 0"/>
       <geometry>
-        <mesh filename="package://racer_model/racer_description/meshes/ZED.dae"/>
+        <box size="${cameraSize} ${cameraSize} ${cameraSize}"/>
       </geometry>
     </visual>
   </link>
+  <gazebo reference="camera">
+    <material>Gazebo/Red</material>
+  </gazebo>
   <joint name="camera_joint" type="fixed">
     <axis xyz="0 1 0" />

Commit message: added mesh

File: ros_ws/src/racer_model/racer_description/urdf/racer.xacro (robot description, xacro)
@@ -3,5 +3,7 @@
   <xacro:include filename="$(find racer_model)/racer_description/urdf/racer_plugins.gazebo" />
   <xacro:include filename="$(find racer_model)/racer_description/urdf/racer_macros.xacro" />
-  <xacro:property name="cameraSize" value="0.05"/>
+  <xacro:property name="cameraSizeL" value="0.03"/>
+  <xacro:property name="cameraSizeB" value="0.03"/>
+  <xacro:property name="cameraSizeH" value="0.17"/>
   <xacro:property name="cameraMass" value="0.1"/>
   <xacro:property name="hokuyoSize" value="0.1"/>
@@ -24,19 +26,16 @@
       </geometry>
     </collision>
-    <visual name='chassis_visual'>
-      <origin xyz="0 0 ${wheel_height/2}" rpy=" 0 0 0"/>
+    <visual>
+      <origin xyz="0 0 0" rpy=" 0 0 0"/>
       <geometry>
-        <box size="${bodySizeL} ${bodySizeB} ${bodySizeH}"/>
+         <mesh filename="package://racer_model/racer_description/meshes/car.dae"/>
       </geometry>
     </visual>
   </link>
-  <gazebo reference="chassis">
-    <material>Gazebo/Green</material>
-  </gazebo>
   <!--  Wheels  -->
-  <wheel  fb="front" lr="left" parent="chassis" translateX="1" translateY="1" flip="90" OffsetY="0.035" />
-  <wheel  fb="back" lr="left" parent="chassis" translateX="-1" translateY="1" flip="90" OffsetY="0.035" />
-  <wheel  fb="front" lr="right" parent="chassis" translateX="1" translateY="-1" flip="90" OffsetY="-0.035" />
-  <wheel  fb="back" lr="right" parent="chassis" translateX="-1" translateY="-1" flip="90" OffsetY="-0.035" />
+  <wheel  fb="front" lr="left" parent="chassis" translateX="1" translateY="1" left="1" OffsetY="0.035" />
+  <wheel  fb="back" lr="left" parent="chassis" translateX="-1" translateY="1" left="1" OffsetY="0.035" />
+  <wheel  fb="front" lr="right" parent="chassis" translateX="1" translateY="-1" left="0" OffsetY="-0.035" />
+  <wheel  fb="back" lr="right" parent="chassis" translateX="-1" translateY="-1" left="0" OffsetY="-0.035" />
   <!-- Steering -->
   <steering_hinge  lr="left" parent="chassis" translateY="1" OffsetY="0.01" />
@@ -47,22 +46,19 @@
       <mass value="${cameraMass}" />
       <origin xyz="0 0 ${wheel_height/2}" rpy="0 0 0"/>
-      <box_inertia m="${cameraMass}" l="${cameraSize}" b="${cameraSize}" h="${cameraSize}" />
+      <box_inertia m="${cameraMass}" l="${cameraSizeL}" b="${cameraSizeB}" h="${cameraSizeH}" />
     </inertial>
     <collision>
-      <origin xyz="0 0 ${wheel_height/2}" rpy="0 0 0"/>
+      <origin xyz="0 0 0" rpy="0 0 0"/>
       <geometry>
-        <box size="${cameraSize} ${cameraSize} ${cameraSize}"/>
+        <box size="${cameraSizeL} ${cameraSizeH} ${cameraSizeB}"/>
       </geometry>
     </collision>
     <visual>
-      <origin xyz="0 0 ${wheel_height/2}" rpy="0 0 0"/>
+      <origin xyz="0 0 0" rpy="0 0 0"/>
       <geometry>
-        <box size="${cameraSize} ${cameraSize} ${cameraSize}"/>
+         <mesh filename="package://racer_model/racer_description/meshes/ZED.dae"/>
       </geometry>
     </visual>
-  </link>
-  <gazebo reference="camera">
-    <material>Gazebo/Red</material>
-  </gazebo>
+  </link>s
   <joint name="camera_joint" type="fixed">
     <axis xyz="0 1 0" />

File: ros_ws/src/racer_model/racer_description/urdf/racer_macros.xacro (robot description, xacro)
@@ -24,13 +24,13 @@
   <property name="base_y_origin_to_wheel_origin" value="0.095" />
   <property name="base_z_origin_to_wheel_origin" value="0" />
-  <xacro:macro name="wheel" params="fb lr parent translateX translateY flip OffsetY">
+  <xacro:macro name="wheel" params="fb lr parent translateX translateY left OffsetY">
     <link name="${lr}_wheel_${fb}">
       <inertial>
         <mass value="${wheel_mass}" />
-        <origin xyz="0 0 0" rpy="${flip*pi/180} 0 0"/>
+        <origin xyz="0 0 0" rpy="${90*pi/180} 0 0"/>
         <cylinder_inertia  m="${wheel_mass}" r="${wheel_radius}" h="${wheel_height}" />
       </inertial>
       <collision>
-        <origin xyz="0 0 0" rpy="${flip*pi/180} 0 0 " />
+        <origin xyz="0 0 0" rpy="${90*pi/180} 0 0 " />
         <geometry>
           <cylinder length="${wheel_height}" radius="${wheel_radius}" />
@@ -38,13 +38,10 @@
       </collision>
       <visual>
-        <origin xyz="0 0 0" rpy="${flip*pi/180} 0  0 " />
+        <origin xyz="0 0 0" rpy="0 0 ${left*pi}" />
         <geometry>
-          <cylinder length="${wheel_height}" radius="${wheel_radius}" />
+          <mesh filename="package://racer_model/racer_description/meshes/wheel.dae"/>
         </geometry>
       </visual>
     </link>
-    <gazebo reference="${lr}_wheel_${fb}">
-      <material>Gazebo/Black</material>
-    </gazebo>
     <joint name="${lr}_wheel_${fb}_hinge" type="continuous">
       <parent link="${parent}"/>

Commit message: gazebo car steering

File: ros_ws/src/racer_model/racer_description/urdf/racer.xacro (robot description, xacro)
@@ -11,4 +11,5 @@
   <xacro:property name="bodySizeH" value="0.1"/>
   <xacro:property name="bodyMass" value="3.5"/>
+  <link name="base_link" />
   <!--  Body  -->
   <link name='chassis'>
@@ -34,12 +35,17 @@
     <material>Gazebo/Green</material>
   </gazebo>
+  <joint name="base_link_joint" type="fixed">
+    <origin xyz="0 0 0.05" rpy="0 0 0" />
+    <parent link="base_link" />
+    <child link="chassis" />
+  </joint>
   <!--  Wheels  -->
-  <wheel  fb="front" lr="left" parent="chassis" translateX="1" translateY="1" flip="90" OffsetY="0.035" />
-  <wheel  fb="back" lr="left" parent="chassis" translateX="-1" translateY="1" flip="90" OffsetY="0.035" />
-  <wheel  fb="front" lr="right" parent="chassis" translateX="1" translateY="-1" flip="90" OffsetY="-0.035" />
-  <wheel  fb="back" lr="right" parent="chassis" translateX="-1" translateY="-1" flip="90" OffsetY="-0.035" />
+  <wheel_front lr="left" parent="left_steering_hinge" translateX="1" translateY="1" flip="90" OffsetY="0.02" />
+  <wheel_front lr="right" parent="right_steering_hinge" translateX="1" translateY="-1" flip="90" OffsetY="-0.02" />
+  <wheel_back lr="left" parent="chassis" translateX="-1" translateY="1" flip="90" OffsetY="0.03" />
+  <wheel_back lr="right" parent="chassis" translateX="-1" translateY="-1" flip="90" OffsetY="-0.03" />
   <!-- Steering -->
-  <steering_hinge  lr="left" parent="chassis" translateY="1" OffsetY="0.01" />
-  <steering_hinge  lr="right" parent="chassis" translateY="-1" OffsetY="-0.01" />
+  <steering_hinge  lr="left" parent="chassis" translateY="1" OffsetY="0.03" />
+  <steering_hinge  lr="right" parent="chassis" translateY="-1" OffsetY="-0.03" />
   <!-- Camera -->
   <link name="camera">
@@ -72,5 +78,5 @@
   </joint>
   <!-- Hokuyo Laser -->
-  <link name="hokuyo">
+  <!-- <link name="hokuyo">
     <inertial>
       <mass value="${hokuyoMass}" />
@@ -96,4 +102,4 @@
     <parent link="chassis"/>
     <child link="hokuyo"/>
-  </joint>
+  </joint> -->
 </robot>

File: ros_ws/src/racer_model/racer_description/urdf/racer_macros.xacro (robot description, xacro)
@@ -17,5 +17,4 @@
               izz="${2*m*(r*r)/3}" />
   </macro>
-  <!-- Wheels -->
   <property name="wheel_radius" value="0.05" />
   <property name="wheel_height" value="0.045" />
@@ -24,6 +23,10 @@
   <property name="base_y_origin_to_wheel_origin" value="0.095" />
   <property name="base_z_origin_to_wheel_origin" value="0" />
-  <xacro:macro name="wheel" params="fb lr parent translateX translateY flip OffsetY">
-    <link name="${lr}_wheel_${fb}">
+  <property name="base_x_sphere_origin_to_wheel_origin" value="0.001" />
+  <property name="base_y_sphere_origin_to_wheel_origin" value="0.001" />
+  <property name="base_z_sphere_origin_to_wheel_origin" value="0" />
+  <!-- Wheels Front-->
+  <xacro:macro name="wheel_front" params="lr parent translateX translateY flip OffsetY">
+    <link name="${lr}_wheel_front">
       <inertial>
         <mass value="${wheel_mass}" />
@@ -32,5 +35,5 @@
       </inertial>
       <collision>
-        <origin xyz="0 0 0" rpy="${flip*pi/180} 0 0 " />
+        <origin xyz="0 ${OffsetY} 0" rpy="${flip*pi/180} 0 0 " />
         <geometry>
           <cylinder length="${wheel_height}" radius="${wheel_radius}" />
@@ -38,5 +41,5 @@
       </collision>
       <visual>
-        <origin xyz="0 0 0" rpy="${flip*pi/180} 0  0 " />
+        <origin xyz="0 ${OffsetY} 0" rpy="${flip*pi/180} 0  0 " />
         <geometry>
           <cylinder length="${wheel_height}" radius="${wheel_radius}" />
@@ -44,21 +47,64 @@
       </visual>
     </link>
-    <gazebo reference="${lr}_wheel_${fb}">
+    <gazebo reference="${lr}_wheel_front">
       <material>Gazebo/Black</material>
     </gazebo>
-    <joint name="${lr}_wheel_${fb}_hinge" type="continuous">
+    <joint name="${lr}_front_wheel_joint" type="continuous">
       <parent link="${parent}"/>
-      <child link="${lr}_wheel_${fb}"/>
-      <origin xyz="${translateX * base_x_origin_to_wheel_origin} ${translateY * base_y_origin_to_wheel_origin + OffsetY} ${base_z_origin_to_wheel_origin}" rpy="0 0 0" />
+      <child link="${lr}_wheel_front"/>
+      <origin xyz="${translateX * base_x_sphere_origin_to_wheel_origin} ${translateY * base_y_sphere_origin_to_wheel_origin} ${base_z_sphere_origin_to_wheel_origin}" rpy="0 0 0" />
       <axis xyz="0 1 0" rpy="0 0 0" />
       <limit effort="10" velocity="100"/>
       <joint_properties damping="0.0" friction="0.0"/>
     </joint>
-    <transmission name="${lr}_wheel_${fb}_transmission" type="SimpleTransmission">
+    <transmission name="${lr}_wheel_front_transmission" type="SimpleTransmission">
       <type>transmission_interface/SimpleTransmission</type>
-      <joint name="${lr}_wheel_${fb}_hinge">
+      <joint name="${lr}_front_wheel_joint">
         <hardwareInterface>hardware_interface/EffortJointInterface</hardwareInterface>
       </joint>
-      <actuator name="${lr}_wheel_${fb}_motor">
+      <actuator name="${lr}_wheel_front_motor">
+        <hardwareInterface>hardware_interface/EffortJointInterface</hardwareInterface>
+        <mechanicalReduction>1</mechanicalReduction>
+      </actuator>
+    </transmission>
+  </xacro:macro>
+  <!-- Wheels Back-->
+  <xacro:macro name="wheel_back" params="lr parent translateX translateY flip OffsetY">
+    <link name="${lr}_wheel_back">
+      <inertial>
+        <mass value="${wheel_mass}" />
+        <origin xyz="0 0 0" rpy="${flip*pi/180} 0 0"/>
+        <cylinder_inertia  m="${wheel_mass}" r="${wheel_radius}" h="${wheel_height}" />
+      </inertial>
+      <collision>
+        <origin xyz="0 ${OffsetY} 0" rpy="${flip*pi/180} 0 0 " />
+        <geometry>
+          <cylinder length="${wheel_height}" radius="${wheel_radius}" />
+        </geometry>
+      </collision>
+      <visual>
+        <origin xyz="0 ${OffsetY} 0" rpy="${flip*pi/180} 0  0 " />
+        <geometry>
+          <cylinder length="${wheel_height}" radius="${wheel_radius}" />
+        </geometry>
+      </visual>
+    </link>
+    <gazebo reference="${lr}_wheel_back">
+      <material>Gazebo/Black</material>
+    </gazebo>
+    <joint name="${lr}_back_wheel_joint" type="continuous">
+      <parent link="${parent}"/>
+      <child link="${lr}_wheel_back"/>
+      <origin xyz="${translateX * base_x_origin_to_wheel_origin} ${translateY * base_y_origin_to_wheel_origin} ${base_z_origin_to_wheel_origin}" rpy="0 0 0" />
+      <axis xyz="0 1 0" rpy="0 0 0" />
+      <limit effort="10" velocity="100"/>
+      <joint_properties damping="0.0" friction="0.0"/>
+    </joint>
+    <transmission name="${lr}_wheel_back_transmission" type="SimpleTransmission">
+      <type>transmission_interface/SimpleTransmission</type>
+      <joint name="${lr}_back_wheel_joint">
+        <hardwareInterface>hardware_interface/EffortJointInterface</hardwareInterface>
+      </joint>
+      <actuator name="${lr}_wheel_back_motor">
         <hardwareInterface>hardware_interface/EffortJointInterface</hardwareInterface>
         <mechanicalReduction>1</mechanicalReduction>
@@ -67,8 +113,8 @@
   </xacro:macro>
   <!-- Steering -->
-  <property name="steering_radius" value="0.025" />
+  <property name="steering_radius" value="0.015" />
   <property name="steering_mass" value="0.07" />
   <xacro:macro name="steering_hinge" params="lr parent translateY OffsetY">
-    <link name="${lr}_steering">
+    <link name="${lr}_steering_hinge">
       <inertial>
         <mass value="${steering_mass}" />
@@ -83,17 +129,17 @@
       </visual>
     </link>
-    <gazebo reference="${lr}_steering">
+    <gazebo reference="${lr}_steering_hinge">
       <material>Gazebo/Grey</material>
     </gazebo>
-    <joint name="${lr}_steering_hinge" type="revolute">
-      <origin xyz="${base_x_origin_to_wheel_origin} ${translateY * base_y_origin_to_wheel_origin + OffsetY} ${base_z_origin_to_wheel_origin}" rpy="0 0 0" />
+    <joint name="${lr}_steering_hinge_joint" type="revolute">
+      <origin xyz="${base_x_origin_to_wheel_origin} ${translateY * base_y_origin_to_wheel_origin + OffsetY} ${ base_z_origin_to_wheel_origin}" rpy="0 0 0" />
       <parent link="${parent}" />
-      <child link="${lr}_steering" />
-      <axis xyz="0 1 0" />
-      <limit lower="-1.0" upper="1.0" effort="10" velocity="100" />
+      <child link="${lr}_steering_hinge" />
+      <axis xyz="0 0 1" />
+      <limit lower="-1.0" upper="1.0" effort="10" velocity="10" />
     </joint>
     <transmission name="${lr}_steering_hinge_transmission" type="SimpleTransmission">
       <type>transmission_interface/SimpleTransmission</type>
-      <joint name="${lr}_steering_hinge">
+      <joint name="${lr}_steering_hinge_joint">
         <hardwareInterface>hardware_interface/EffortJointInterface</hardwareInterface>
       </joint>

Commit message: Control car with keyboard or let it drive autonomously

File: ros_ws/src/racer_model/racer_description/urdf/racer.xacro (robot description, xacro)
@@ -1,6 +1,6 @@
 <?xml version='1.0'?>
 <robot name="myrobot" xmlns:xacro="http://www.ros.org/wiki/xacro">
-  <xacro:include filename="$(find racer_model)/racer_description/urdf/racer_plugins.gazebo" />
-  <xacro:include filename="$(find racer_model)/racer_description/urdf/racer_macros.xacro" />
+  <xacro:include filename="$(find racer_description)/urdf/racer_plugins.gazebo" />
+  <xacro:include filename="$(find racer_description)/urdf/racer_macros.xacro" />
   <xacro:property name="cameraSizeL" value="0.03"/>
   <xacro:property name="cameraSizeB" value="0.03"/>
@@ -29,5 +29,5 @@
       <origin xyz="0 0 0" rpy=" 0 0 0"/>
       <geometry>
-         <mesh filename="package://racer_model/racer_description/meshes/car.dae"/>
+         <mesh filename="package://racer_description/meshes/car.dae"/>
       </geometry>
     </visual>
@@ -57,5 +57,5 @@
       <origin xyz="0 0 0" rpy="0 0 0"/>
       <geometry>
-         <mesh filename="package://racer_model/racer_description/meshes/ZED.dae"/>
+         <mesh filename="package://racer_description/meshes/ZED.dae"/>
       </geometry>
     </visual>
@@ -83,5 +83,5 @@
       <origin xyz="0 0 ${wheel_height/2}" rpy="0 0 0"/>
       <geometry>
-        <mesh filename="package://racer_model/racer_description/meshes/hokuyo.dae"/>
+        <mesh filename="package://racer_description/meshes/hokuyo.dae"/>
       </geometry>
     </visual>

File: ros_ws/src/racer_model/racer_description/urdf/racer_macros.xacro (robot description, xacro)
@@ -40,5 +40,5 @@
         <origin xyz="0 0 0" rpy="0 0 ${left*pi}" />
         <geometry>
-          <mesh filename="package://racer_model/racer_description/meshes/wheel.dae"/>
+          <mesh filename="package://racer_description/meshes/wheel.dae"/>
         </geometry>
       </visual>
