Commit message: test params

File: ros_ws/src/simulation/racer_description/urdf/racer.xacro (robot description, xacro)
@@ -10,5 +10,5 @@
   <xacro:property name="hokuyoMass" value="0.1"/>
   <xacro:property name="bodySizeL" value="0.49"/>
-  <xacro:property name="bodySizeB" value="0.18"/>
+  <xacro:property name="bodySizeB" value="0.2315"/>
   <xacro:property name="bodySizeH" value="0.1"/>
   <xacro:property name="bodyMass" value="3.5"/>
